Commit message: Updated files

File: nav2/sam_bot_description/src/description/sam_bot_description.urdf (robot description, URDF)
Before this commit: robot sam_bot, 4 links, 3 joints
Links:
- removed link imu_link
- added link zed_camera_link; visual box size=0.04 0.2 0.035
Joints:
- removed joint imu_joint
- added joint zed_camera_joint: type fixed, parent base_link, child zed_camera_link, origin xyz=0.23 0 0 rpy=0 0 0

Commit message: Working autonomy

File: nav2/sam_bot_description/src/description/sam_bot_description.urdf (robot description, URDF)
Before this commit: robot sam_bot, 4 links, 3 joints
Links:
- link lidar_link: geometry visual cylinder length=${lidar_height} radius=${lidar_radius}
- link zed_camera_link: geometry visual box size=${zed_length} ${zed_width} ${zed_height}
Joints:
- joint base_joint: origin xyz=0.0 0.0 ${-(base_height / 2)} rpy=0 0 0 -> xyz=0.0 0.0 ${-(wheel_radius+wheel_zoff)} rpy=0 0 0
- joint lidar_joint: origin xyz=0 0 0.12 rpy=0 0 0 -> xyz=${(base_length / 2) + (lidar_radius / 2) + 0.030} 0 ${(base_height / 2) - 0.120 + (lidar_height / 2)} rpy=0 0 ${pi}
- joint zed_camera_joint: origin xyz=0.23 0 0 rpy=0 0 0 -> xyz=${(base_length / 2) - (zed_length / 2)} 0 ${(base_height / 2) + (zed_height / 2)} rpy=0 0 0

Commit message: Autonomy code gnss - Needs full test

File: nav2/sam_bot_description/src/description/sam_bot_description.urdf (robot description, URDF)
Before this commit: robot sam_bot, 4 links, 3 joints
Links:
- added link gnss_moving_base_link; visual cylinder length=${gnss_moving_base_height} radius=${gnss_moving_base_radius}
- added link gnss_moving_rover_link; visual cylinder length=${gnss_moving_rover_height} radius=${gnss_moving_rover_radius}
Joints:
- added joint gnss_moving_base_joint: type fixed, parent base_link, child gnss_moving_base_link, origin xyz=${0.127 - (base_length / 2)} ${0.0251 - (base_width / 2)} ${(base_height / 2) + (gnss_moving_base_height / 2)} rpy=0 0 0
- added joint gnss_moving_rover_joint: type fixed, parent base_link, child gnss_moving_rover_link, origin xyz=${(base_length / 2) - 0.127} ${(base_width / 2) - 0.0251} ${(base_height / 2) + (gnss_moving_rover_height / 2)} rpy=0 0 0

Commit message: Working on automony

File: nav2/sam_bot_description/src/description/sam_bot_description.urdf (robot description, URDF)
Before this commit: robot sam_bot, 6 links, 5 joints
Joints:
- joint gnss_moving_base_joint: origin xyz=${0.127 - (base_length / 2)} ${0.0251 - (base_width / 2)} ${(base_height / 2) + (gnss_moving_base_height / 2)} rpy=0 0 0 -> xyz=${0.127 - (base_length / 2)} ${0.057 - (base_width / 2)} ${(base_height / 2) + (gnss_moving_base_height / 2)} rpy=0 0 0

Commit message: Working working mapviz

File: nav2/sam_bot_description/src/description/sam_bot_description.urdf (robot description, URDF)
Before this commit: robot sam_bot, 6 links, 5 joints
Joints:
- joint gnss_moving_base_joint: origin xyz=${0.127 - (base_length / 2)} ${0.057 - (base_width / 2)} ${(base_height / 2) + (gnss_moving_base_height / 2)} rpy=0 0 0 -> xyz=${0.127 - (base_length / 2)} ${0.0251 - (base_width / 2)} ${(base_height / 2) + (gnss_moving_base_height / 2)} rpy=0 0 0
